Commit message: Changed the mass of the drone from 27 grams to 33 grams

File: gym_pybullet_drones/assets/cf2x.urdf (robot description, URDF)
Before this commit: robot cf2, 6 links, 5 joints
Links:
- link base_link: mass 0.027 -> 0.033

Commit message: Base training 3: drone mass: 0.027 kg initial position: [0 0 0] initial attitude: [0 0 0] pybullet frequency: 240 control frequency: 30 batch size: 128 parallel environments: 4

File: gym_pybullet_drones/assets/cf2x.urdf (robot description, URDF)
Before this commit: robot cf2, 6 links, 5 joints
Links:
- link base_link: mass 0.033 -> 0.027
